File: pcb/nabu-sio.kicad_pcb (KiCad board)
At the start: 2 copper layers, 119.4 x 58.4 mm, 34 parts, among them IC1 CTC-DIP-28, IC2 SIO1-DIP-40, J1 NABU Extension Slot, J2 Conn_02x05_Odd_Even, J3 Conn_02x05_Odd_Even, J4 PORT A TTL, J5 PORT B TTL, U1 MAX232, U2 MAX232, U3 MAX232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

Commit message: Version 0.1 sent to production
Other:
- board text added: "Version: 0.1"
Changed lines of the file:
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@@
       (outputformat 1)
       (mirror false)
-      (drillshape 1)
+      (drillshape 0)
       (scaleselection 1)
-      (outputdirectory "")
+      (outputdirectory "gerber/")
     )
   )
@@
   (gr_arc (start 202.038949 64.243949) (mid 203.835 64.987898) (end 204.578949 66.783949) (layer "Edge.Cuts") (width 0.1))
   (gr_arc (start 169.018949 115.043949) (mid 169.762898 113.247898) (end 171.558949 112.503949) (layer "Edge.Cuts") (width 0.1))
+  (gr_text "Version: 0.1" (at 156.972 110.998) (layer "F.Cu")
+    (effects (font (size 1 1) (thickness 0.15)))
+  )
   (gr_text "4×1µF" (at 183.896 78.232) (layer "B.SilkS")
     (effects (font (size 1 1) (thickness 0.15)) (justify mirror))

Commit message: Fix some labels
Parts:
- IC1: value CTC-DIP-28 -> Z80 CTC
- IC2: value SIO1-DIP-40 -> Z80 SIO
- J2: value Conn_02x05_Odd_Even -> PORT A RS232
- J3: value Conn_02x05_Odd_Even -> PORT B RS232
Changed lines of the file:
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@@
       (effects (font (size 1 1) (thickness 0.15)))
     )
-    (fp_text value "SIO1-DIP-40" (at 6.438949 34.176051 180) (layer "F.SilkS")
+    (fp_text value "Z80 SIO" (at 6.438949 34.176051 180) (layer "F.SilkS")
       (effects (font (size 1 1) (thickness 0.15)))
     )
@@
       (effects (font (size 1 1) (thickness 0.15)))
     )
-    (fp_text value "Conn_02x05_Odd_Even" (at 5.655 12.43) (layer "F.SilkS")
+    (fp_text value "PORT A RS232" (at 5.362051 12.967051) (layer "F.SilkS")
       (effects (font (size 1 1) (thickness 0.15)))
     )
@@
       (effects (font (size 1 1) (thickness 0.15)))
     )
-    (fp_text value "CTC-DIP-28" (at 6.438949 26.551051 180) (layer "F.SilkS")
+    (fp_text value "Z80 CTC" (at 6.438949 26.551051 180) (layer "F.SilkS")
       (effects (font (size 1 1) (thickness 0.15)))
     )
@@
       (effects (font (size 1 1) (thickness 0.15)))
     )
-    (fp_text value "PORT A TTL" (at -2.431051 6.241051 180) (layer "F.SilkS")
+    (fp_text value "PORT A TTL" (at -2.685051 6.241051 180) (layer "F.SilkS")
       (effects (font (size 1 1) (thickness 0.15)))
     )
@@
       (effects (font (size 1 1) (thickness 0.15)))
     )
-    (fp_text value "Conn_02x05_Odd_Even" (at 5.655 12.43) (layer "F.SilkS")
+    (fp_text value "PORT B RS232" (at 5.489051 12.967051) (layer "F.SilkS")
       (effects (font (size 1 1) (thickness 0.15)))
     )
@@
       (effects (font (size 1 1) (thickness 0.15)))
     )
-    (fp_text value "PORT B TTL" (at -2.431051 6.241051 180) (layer "F.SilkS")
-      (effects (font (size 1 1) (thickness 0.15)))
-    )
+    (fp_text value "PORT B TTL" (at -2.685051 6.241051 180) (layer "F.SilkS")
+      (effects (font (size 1 1) (thickness 0.15)))
+    )

Commit message: Various fixes
Parts:
- IC1: value Z80 CTC -> Z80A CTC
- IC2: value Z80 SIO -> Z80A SIO
Other:
- board text added: "Version: 0.2"
- board text removed: "Version: 0.1"
Changed lines of the file:
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@@
   (net 97 "unconnected-(J2-Pad10)")
   (net 98 "unconnected-(J3-Pad10)")
-  (net 99 "Net-(U5-Pad8)")
+  (net 99 "Net-(U4-Pad13)")
   (footprint "Connector_PinSocket_2.54mm:PinSocket_1x30_P2.54mm_Vertical" (layer "F.Cu")
     (at 163.958949 119.533949 -90)
@@
     )
     (fp_text user "~{M1}" (at -3.328949 2.541949 -90 unlocked) (layer "B.SilkS")
-      (effects (font (size 1 1) (thickness 0.15)))
+      (effects (font (size 1 1) (thickness 0.15)) (justify mirror))
     )
     (fp_text user "D3" (at -3.328949 45.721949 -90 unlocked) (layer "B.SilkS")
-      (effects (font (size 1 1) (thickness 0.15)))
+      (effects (font (size 1 1) (thickness 0.15)) (justify mirror))
     )
     (fp_text user "A2" (at -3.328949 17.781949 -90 unlocked) (layer "B.SilkS")
-      (effects (font (size 1 1) (thickness 0.15)))
+      (effects (font (size 1 1) (thickness 0.15)) (justify mirror))
     )
     (fp_text user "D5" (at -3.328949 50.801949 -90 unlocked) (layer "B.SilkS")
-      (effects (font (size 1 1) (thickness 0.15)))
+      (effects (font (size 1 1) (thickness 0.15)) (justify mirror))
     )
     (fp_text user "A0" (at -3.328949 12.701949 -90 unlocked) (layer "B.SilkS")
-      (effects (font (size 1 1) (thickness 0.15)))
+      (effects (font (size 1 1) (thickness 0.15)) (justify mirror))
     )
     (fp_text user "~{INT}" (at -3.328949 0.001949 -90 unlocked) (layer "B.SilkS")
-      (effects (font (size 1 1) (thickness 0.15)))
+      (effects (font (size 1 1) (thickness 0.15)) (justify mirror))
     )
     (fp_text user "-12V" (at -3.328949 73.661949 -90 unlocked) (layer "B.SilkS")
-      (effects (font (size 1 1) (thickness 0.15)))
+      (effects (font (size 1 1) (thickness 0.15)) (justify mirror))
     )
     (fp_text user "~{WAIT}" (at -3.328949 33.021949 -90 unlocked) (layer "B.SilkS")
-      (effects (font (size 1 1) (thickness 0.15)))
+      (effects (font (size 1 1) (thickness 0.15)) (justify mirror))
     )
     (fp_text user "D7" (at -3.328949 55.881949 -90 unlocked) (layer "B.SilkS")
-      (effects (font (size 1 1) (thickness 0.15)))
+      (effects (font (size 1 1) (thickness 0.15)) (justify mirror))
     )
     (fp_text user "A3" (at -3.328949 20.321949 -90 unlocked) (layer "B.SilkS")
-      (effects (font (size 1 1) (thickness 0.15)))
+      (effects (font (size 1 1) (thickness 0.15)) (justify mirror))
     )
     (fp_text user "GND" (at -3.328949 68.581949 -90 unlocked) (layer "B.SilkS")
-      (effects (font (size 1 1) (thickness 0.15)))
+      (effects (font (size 1 1) (thickness 0.15)) (justify mirror))
     )
     (fp_text user "~{WR}" (at -3.328949 25.401949 -90 unlocked) (layer "B.SilkS")
-      (effects (font (size 1 1) (thickness 0.15)))
+      (effects (font (size 1 1) (thickness 0.15)) (justify mirror))
     )
     (fp_text user "~{IORQ}" (at -3.328949 30.481949 -90 unlocked) (layer "B.SilkS")
-      (effects (font (size 1 1) (thickness 0.15)))
+      (effects (font (size 1 1) (thickness 0.15)) (justify mirror))
     )
     (fp_text user "GND" (at -3.328949 63.501949 -90 unlocked) (layer "B.SilkS")
-      (effects (font (size 1 1) (thickness 0.15)))
+      (effects (font (size 1 1) (thickness 0.15)) (justify mirror))
     )
     (fp_text user "~{RESET}" (at -3.328949 35.561949 -90 unlocked) (layer "B.SilkS")
-      (effects (font (size 1 1) (thickness 0.15)))
+      (effects (font (size 1 1) (thickness 0.15)) (justify mirror))
     )
     (fp_text user "D2" (at -3.328949 43.181949 -90 unlocked) (layer "B.SilkS")
-      (effects (font (size 1 1) (thickness 0.15)))
+      (effects (font (size 1 1) (thickness 0.15)) (justify mirror))
     )
     (fp_text user "+5V" (at -3.328949 58.421949 -90 unlocked) (layer "B.SilkS")
-      (effects (font (size 1 1) (thickness 0.15)))
+      (effects (font (size 1 1) (thickness 0.15)) (justify mirror))
     )
     (fp_text user "AUDIO" (at -3.328949 7.621949 -90 unlocked) (layer "B.SilkS")
-      (effects (font (size 1 1) (thickness 0.15)))
+      (effects (font (size 1 1) (thickness 0.15)) (justify mirror))
     )
     (fp_text user "D4" (at -3.328949 48.261949 -90 unlocked) (layer "B.SilkS")
-      (effects (font (size 1 1) (thickness 0.15)))
+      (effects (font (size 1 1) (thickness 0.15)) (justify mirror))
     )
     (fp_text user "~{CS}" (at -3.328949 10.161949 -90 unlocked) (layer "B.SilkS")
-      (effects (font (size 1 1) (thickness 0.15)))
+      (effects (font (size 1 1) (thickness 0.15)) (justify mirror))
     )
     (fp_text user "3.58" (at -3.328949 5.081949 -90 unlocked) (layer "B.SilkS")
-      (effects (font (size 1 1) (thickness 0.15)))
+      (effects (font (size 1 1) (thickness 0.15)) (justify mirror))
     )
     (fp_text user "D0" (at -3.328949 38.101949 -90 unlocked) (layer "B.SilkS")
-      (effects (font (size 1 1) (thickness 0.15)))
+      (effects (font (size 1 1) (thickness 0.15)) (justify mirror))
     )
     (fp_text user "+5V" (at -3.328949 60.961949 -90 unlocked) (layer "B.SilkS")
-      (effects (font (size 1 1) (thickness 0.15)))
+      (effects (font (size 1 1) (thickness 0.15)) (justify mirror))
     )
     (fp_text user "+12V" (at -3.328949 71.121949 -90 unlocked) (layer "B.SilkS")
-      (effects (font (size 1 1) (thickness 0.15)))
+      (effects (font (size 1 1) (thickness 0.15)) (justify mirror))
     )
     (fp_text user "A1" (at -3.328949 15.241949 -90 unlocked) (layer "B.SilkS")
-      (effects (font (size 1 1) (thickness 0.15)))
+      (effects (font (size 1 1) (thickness 0.15)) (justify mirror))
     )
     (fp_text user "D6" (at -3.328949 53.341949 -90 unlocked) (layer "B.SilkS")
-      (effects (font (size 1 1) (thickness 0.15)))
+      (effects (font (size 1 1) (thickness 0.15)) (justify mirror))
     )
     (fp_text user "~{RD}" (at -3.328949 27.941949 -90 unlocked) (layer "B.SilkS")
-      (effects (font (size 1 1) (thickness 0.15)))
+      (effects (font (size 1 1) (thickness 0.15)) (justify mirror))
     )
     (fp_text user "1.79" (at -3.328949 22.861949 -90 unlocked) (layer "B.SilkS")
-      (effects (font (size 1 1) (thickness 0.15)))
+      (effects (font (size 1 1) (thickness 0.15)) (justify mirror))
     )
     (fp_text user "GND" (at -3.328949 66.041949 -90 unlocked) (layer "B.SilkS")
-      (effects (font (size 1 1) (thickness 0.15)))
+      (effects (font (size 1 1) (thickness 0.15)) (justify mirror))
     )
     (fp_text user "D1" (at -3.328949 40.641949 -90 unlocked) (layer "B.SilkS")
-      (effects (font (size 1 1) (thickness 0.15)))
+      (effects (font (size 1 1) (thickness 0.15)) (justify mirror))
     )
     (fp_text user "-12V" (at -4.6 73.679507 -90 unlocked) (layer "F.SilkS")
@@
       (effects (font (size 1 1) (thickness 0.15)))
     )
-    (fp_text value "Z80 SIO" (at 6.438949 34.176051 180) (layer "F.SilkS")
+    (fp_text value "Z80A SIO" (at 6.438949 34.176051 180) (layer "F.SilkS")
       (effects (font (size 1 1) (thickness 0.15)))
     )
@@
       (effects (font (size 1 1) (thickness 0.15)))
     )
-    (fp_text value "Z80 CTC" (at 6.438949 26.551051 180) (layer "F.SilkS")
+    (fp_text value "Z80A CTC" (at 6.438949 26.551051 180) (layer "F.SilkS")
       (effects (font (size 1 1) (thickness 0.15)))
     )
@@
       (net 24 "/A3") (pintype "input"))
     (pad "13" smd roundrect (at 2.69 2.54 180) (size 1.6 0.6) (layers "B.Cu" "B.Paste" "B.Mask") (roundrect_rratio 0.25)
-      (net 99 "Net-(U5-Pad8)") (pintype "input"))
+      (net 99 "Net-(U4-Pad13)") (pintype "input"))
     (pad "14" smd roundrect (at 2.69 3.81 180) (size 1.6 0.6) (layers "B.Cu" "B.Paste" "B.Mask") (roundrect_rratio 0.25)
       (net 65 "VCC") (pinfunction "VCC") (pintype "power_in"))
@@
       (net 66 "GND") (pinfunction "GND") (pintype "power_in"))
     (pad "8" smd roundrect (at 2.671453 -3.744974 180) (size 1.6 0.6) (layers "B.Cu" "B.Paste" "B.Mask") (roundrect_rratio 0.25)
-      (net 99 "Net-(U5-Pad8)") (pintype "output"))
+      (net 99 "Net-(U4-Pad13)") (pintype "output"))
     (pad "9" smd roundrect (at 2.69 -2.54 180) (size 1.6 0.6) (layers "B.Cu" "B.Paste" "B.Mask") (roundrect_rratio 0.25)
       (net 23 "/A2") (pintype "input"))
@@
   (gr_arc (start 202.038949 64.243949) (mid 203.835 64.987898) (end 204.578949 66.783949) (layer "Edge.Cuts") (width 0.1))
   (gr_arc (start 169.018949 115.043949) (mid 169.762898 113.247898) (end 171.558949 112.503949) (layer "Edge.Cuts") (width 0.1))
-  (gr_text "Version: 0.1" (at 156.972 110.998) (layer "F.Cu")
-    (effects (font (size 1 1) (thickness 0.15)))
-  )
   (gr_text "4×1µF" (at 183.896 78.232) (layer "B.SilkS")
     (effects (font (size 1 1) (thickness 0.15)) (justify mirror))
@@
     (effects (font (size 1 1) (thickness 0.15)) (justify mirror))
   )
+  (gr_text "Version: 0.2" (at 156.972 110.998) (layer "F.SilkS")
+    (effects (font (size 1 1) (thickness 0.15)))
+  )
   (gr_text "nabu-sio" (at 162.56 103.632) (layer "F.SilkS")
