File: pcb/nabu-sio.kicad_sch (KiCad schematic)
At the start: 34 parts, among them IC1 CTC-DIP-28, IC2 SIO1-DIP-40, J1 NABU Extension Slot, J2 Conn_02x05_Odd_Even, J3 Conn_02x05_Odd_Even, J4 PORT A TTL, J5 PORT B TTL, U1 MAX232, U2 MAX232, U3 MAX232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

Commit message: Various fixes
Parts:
- IC1: value CTC-DIP-28 -> Z80A CTC
- IC2: value SIO1-DIP-40 -> Z80A SIO
- J2: value Conn_02x05_Odd_Even -> PORT A RS232
- J3: value Conn_02x05_Odd_Even -> PORT B RS232
Changed lines of the file:
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@@
   (symbol (lib_id "Connector_Generic:Conn_02x05_Odd_Even") (at 323.215 115.57 0) (unit 1)
     (in_bom yes) (on_board yes) (fields_autoplaced)
-    (property "Reference" "J2" (id 0) (at 324.485 103.505 0))
-    (property "Value" "Conn_02x05_Odd_Even" (id 1) (at 324.485 106.045 0))
+    (property "Reference" "J2" (id 0) (at 324.485 104.14 0))
+    (property "Value" "PORT A RS232" (id 1) (at 324.485 106.68 0))
     (property "Footprint" "Connector_PinHeader_2.54mm:PinHeader_2x05_P2.54mm_Horizontal" (id 2) (at 323.215 115.57 0)
       (effects (font (size 1.27 1.27)) hide)
@@
       (effects (font (size 1.27 1.27)) (justify left))
     )
-    (property "Value" "CTC-DIP-28" (id 1) (at 217.9194 50.8 0)
+    (property "Value" "Z80A CTC" (id 1) (at 217.9194 50.8 0)
       (effects (font (size 1.27 1.27)) (justify left))
     )
@@
     (in_bom yes) (on_board yes) (fields_autoplaced)
     (property "Reference" "J3" (id 0) (at 324.485 156.21 0))
-    (property "Value" "Conn_02x05_Odd_Even" (id 1) (at 324.485 158.75 0))
+    (property "Value" "PORT B RS232" (id 1) (at 324.485 158.75 0))
     (property "Footprint" "Connector_PinHeader_2.54mm:PinHeader_2x05_P2.54mm_Horizontal" (id 2) (at 323.215 168.275 0)
       (effects (font (size 1.27 1.27)) hide)
@@
   (symbol (lib_id "Zilog_Z80_Peripherals:SIO1-DIP-40") (at 208.28 123.19 0) (unit 1)
     (in_bom yes) (on_board yes) (fields_autoplaced)
-    (property "Reference" "IC2" (id 0) (at 217.9194 117.475 0)
-      (effects (font (size 1.27 1.27)) (justify left))
-    )
-    (property "Value" "SIO1-DIP-40" (id 1) (at 217.9194 120.015 0)
+    (property "Reference" "IC2" (id 0) (at 217.9194 118.11 0)
+      (effects (font (size 1.27 1.27)) (justify left))
+    )
+    (property "Value" "Z80A SIO" (id 1) (at 217.9194 120.65 0)
       (effects (font (size 1.27 1.27)) (justify left))
     )
@@
     )
     (path "/2ecc2232-ba5b-4a4a-aa38-b74b0c1a1b6d"
-      (reference "IC1") (unit 1) (value "CTC-DIP-28") (footprint "Package_DIP:DIP-28_W15.24mm_LongPads")
+      (reference "IC1") (unit 1) (value "Z80A CTC") (footprint "Package_DIP:DIP-28_W15.24mm_LongPads")
     )
     (path "/ef00d8f1-853d-4e7c-9780-fa343a73cb15"
-      (reference "IC2") (unit 1) (value "SIO1-DIP-40") (footprint "Package_DIP:DIP-40_W15.24mm_LongPads")
+      (reference "IC2") (unit 1) (value "Z80A SIO") (footprint "Package_DIP:DIP-40_W15.24mm_LongPads")
     )
     (path "/b0249235-4bd0-4b35-86ae-b69361039425"
@@
     )
     (path "/124337a5-5555-400f-9c16-3805b43b214b"
-      (reference "J2") (unit 1) (value "Conn_02x05_Odd_Even") (footprint "Connector_PinHeader_2.54mm:PinHeader_2x05_P2.54mm_Horizontal")
+      (reference "J2") (unit 1) (value "PORT A RS232") (footprint "Connector_PinHeader_2.54mm:PinHeader_2x05_P2.54mm_Horizontal")
     )
     (path "/c9976af9-d8c0-4fbc-a965-0fab478ccc50"
-      (reference "J3") (unit 1) (value "Conn_02x05_Odd_Even") (footprint "Connector_PinHeader_2.54mm:PinHeader_2x05_P2.54mm_Horizontal")
+      (reference "J3") (unit 1) (value "PORT B RS232") (footprint "Connector_PinHeader_2.54mm:PinHeader_2x05_P2.54mm_Horizontal")
     )
     (path "/8283e37a-d5af-41b2-a8d6-2f8dada0ec32"
